File: pcb_gift.brd (EAGLE design)
At the start: 37 x 51 mm, 19 parts, among them U1 ATTINY84, U2 BRM-2A18RA

Commit message: updated code for new revision and cleaned things up
- added bom
- updated firmware for this version
- firmware has deeper sleep mode
- added scripts to compile/upload to board
- added .gitignore
- updated readme
- added images of the final board schematic, and component locations
Parts:
- R14: value 680 -> 2k
- R3: value 1.2k -> 1k
Changed lines of the file:
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@@
 <element name="R1" library="resistor" package="R0805" value="560" x="2.8" y="40.25" rot="MR90"/>
 <element name="R2" library="resistor" package="R0805" value="820" x="29.6" y="46.2" rot="MR180"/>
-<element name="R3" library="resistor" package="R0805" value="1.2k" x="31.9" y="12.4" rot="MR270"/>
-<element name="R14" library="resistor" package="R0805" value="680" x="4.9" y="13.2" rot="MR270"/>
+<element name="R3" library="resistor" package="R0805" value="1k" x="31.9" y="12.4" rot="MR270"/>
+<element name="R14" library="resistor" package="R0805" value="2k" x="4.9" y="13.2" rot="MR270"/>
 <element name="D5" library="widget" package="LED5MM_SIDE" value="LED5MM_SIDE" x="15" y="41.9" smashed="yes">
 <attribute name="NAME" x="18.175" y="42.4334" size="1.27" layer="25" font="vector" ratio="10"/>
